File: front_panel/front_panel.kicad_pcb (KiCad board)
At the start: 2 copper layers, 46 parts, among them J1 Conn_01x03_Socket, J10 Conn_01x02_Socket, J11 Conn_01x02_Socket, J12 Conn_01x02_Socket, J13 Conn_01x02_Socket, J14 Conn_01x02_Socket, J15 Conn_01x02_Socket, J16 Conn_01x02_Socket, J17 Conn_01x02_Socket, J18 Conn_01x02_Socket, J19 Conn_01x03_Pin, J2 Conn_01x02_Socket, J20 Conn_01x02_Socket, J21 Conn_01x03_Pin, J3 Conn_01x02_Socket, J5 Conn_01x02_Socket, J6 Conn_01x05_Pin, J7 Conn_01x02_Socket, J8 Conn_01x02_Socket, J9 Conn_01x02_Socket, Q1 DMN3023L, Q2 DMN3023L, SW2 SW_MEC_5G, U1 NCS21804, U10 MCP9700x-ETT, U11 MCP33141D-05, U2 LM4040DBZ-4.1, U3 NCS21804, U4 CD74HC4067M, U5 DAC60501, U6 MIC5504-1.8YM5, U7 BP, U8 CD74HC4067M, U9 MCP9700x-ETT

Commit message: Konačno PCB za BJT modul je počeo.
Parts:
- added SW1: RotaryEncoder_Switch, Rotary_Encoder:RotaryEncoder_Alps_EC12E-Switch_Vertical_H20mm, F.Cu at (105.5, 50.1)
- added SW3: SW_MEC_5G, Button_Switch_SMD:SW_SPST_B3S-1000, F.Cu at (109.0, 64.5)
- moved U11 45.8 mm to (118.2, 62.6)
Connections:
- SW2 pad 1: Net-(SW2-A-Pad1) -> 5V
- SW2 pad 2: Net-(SW2-A-Pad1) -> 5V
- U11 pad 6: unconnected-(U11-CNVST-Pad6) -> CNVST
- U11 pad 7: unconnected-(U11-SDO-Pad7) -> SPI1_MISO
- U11 pad 8: unconnected-(U11-SCLK-Pad8) -> SPI1_CLK
- U11 pad 9: unconnected-(U11-SDI-Pad9) -> 3.3V
- U5 pad 5: unconnected-(U5-SPI2C-Pad5) -> 0
- U5 pad 6: unconnected-(U5-SCLK-Pad6) -> SPI1_CLK
- U5 pad 7: unconnected-(U5-SDA-Pad7) -> SPI1_MOSI
- U7 pad 5V: unconnected-(U7-Pad5V) -> 5V
- U7 pad G: unconnected-(U7-GND-PadG) -> 0
- U7 pad PA0: unconnected-(U7-PadPA0) -> OUTPUT3
- U7 pad PA1: unconnected-(U7-PadPA1) -> INPUT0
- U7 pad PA10: unconnected-(U7-PadPA10) -> B0
- U7 pad PA15: unconnected-(U7-PadPA15) -> B0
- U7 pad PA2: unconnected-(U7-PadPA2) -> INPUT1
- U7 pad PA3: unconnected-(U7-PadPA3) -> INPUT2
- U7 pad PA4: OUTPUT0 -> INPUT3
- U7 pad PA5: OUTPUT1 -> SPI1_CLK
- U7 pad PA6: OUTPUT2 -> SPI1_MISO
- U7 pad PA7: OUTPUT3 -> CNVST
- U7 pad PA8: unconnected-(U7-PadPA8) -> B0
- U7 pad PA9: unconnected-(U7-PadPA9) -> B0
- U7 pad PB0: INPUT0 -> B0
- U7 pad PB1: INPUT1 -> B0
- U7 pad PB10: INPUT2 -> B0
- U7 pad PB11: INPUT3 -> unconnected-(U7-PadPB11)
- U7 pad PB12: unconnected-(U7-PadPB12) -> B0
- U7 pad PB13: unconnected-(U7-PadPB13) -> SPI1_CLK
- U7 pad PB14: unconnected-(U7-PadPB14) -> ~{SYNC}
- U7 pad PB15: unconnected-(U7-PadPB15) -> SPI1_MOSI
- U7 pad PC13: unconnected-(U7-PadPC13) -> OUTPUT0
- U7 pad PC14: unconnected-(U7-PadPC14) -> OUTPUT1
- U7 pad PC15: unconnected-(U7-PadPC15) -> OUTPUT2
